Commit message: Throw planner v3: planning module, matched-t windup, evade flip-brake
End-to-end pipeline replacing the hand-tuned throw choreography:

src/planner.py (new)
  Grid+Pareto throw planner. Sweeps (release_x, vz) for given drone/
  ball/room params, applies hard constraints (apex below ceiling, thrust
  within max, tilt within max, backup in play area, ball reaches catcher,
  evade-brake distance fits in play area), returns Pareto frontier on
  (arrival_KE ↓, min_margin ↑). plan() picks by `prefer=` policy:
  pareto / min_ke / max_throw / max_margin. diagnose_infeasibility()
  walks constraints to explain why no plan was found.

src/controller.py (new) + src/drone.py (refactored)
  Pulled the cascaded position+attitude controller out of Drone.step()
  into a CascadeController dataclass. Drone now stitches state queries
  → controller → applyExternal*. Behavior preserved exactly. max_tilt_deg
  is a controller field, so we can temporarily flip it to 90° in evade.

src/main.py
  Replaces hardcoded throw geometry with one plan_throw() call. Windup
  loop follows a matched-t trajectory where pos_target IS the integral
  of vel_target — eliminates the position-vs-velocity contradiction
  that was making the controller undershoot vz. After release, the
  controller's max_tilt_deg is bumped to 90° so the drone can flip-brake
  (full thrust horizontal in -x), matching the planner's brake_decel
  assumption (max_thrust/m_drone ≈ 21.8 m/s²).

  No-overlap play areas: each drone owns half the room (centerline at
  x=0). Sport-like, prevents poaching. Default plan policy is "max_throw"
  (flat fastball) instead of min_ke (high arc / drop).

  Camera repositioned for the wider 12 m room (side-spectator view from
  inside the arena, 90° FOV). Static magenta marker shows the planner-
  committed release_pos so the moving trajectory carrot doesn't look
  like re-optimization.

src/world.py
  Walls and ceiling are now collision-only (no visual). PyBullet's
  tinyrenderer doesn't blend alpha properly, so transparent walls were
  rendering opaque and blocking the camera. Visual reference for the
  arena now comes from the play-area wireframe outlines.

docs/throw_planning.md (new, ~370 lines)
  Full math: ballistic targeting, drone trajectory generation, the
  matched-t single ramp insight (backup_pos = release_pos − ½·vel·t_ramp),
  free variables, hard constraints, Pareto frontier, grid+Pareto pipeline,
  multi-phase considerations. Cites Mellinger/Kumar, Hehn/D'Andrea, FMA,
  TossingBot.

scripts/plot_windup.py (new)
  Plots planned vs actual drone trajectory through windup (pos x/z and
  vel x/z). Made debugging the cascade-vs-plan mismatch tractable.

Verification: end-to-end demo runs cleanly. Throw lands at catcher with
release vel within ~5% of plan. Catch + cube pickup + lift all complete
within 18 s.

Co-Authored-By: Claude Opus 4.7 (1M context) <noreply@anthropic.com>

File: assets/quadrotor.urdf (robot description, URDF)
Before this commit: robot quadrotor, 5 links, 4 joints
Links:
- link base_link: mass 0.5 -> 0.546

Commit message: WIP: 2-link arm — URDF, joint discovery, CoM compensation, stationary throw skeleton
This is checkpoint progress on the bowling-style arm work (plan in
/home/cosmopal/.claude/plans/next-up-is-the-quiet-dusk.md). Hover, arm
extension, ball-grasp-at-EE all work. Throw fires but mechanics need
significant tuning. Committing now to capture progress before further work.

assets/quadrotor.urdf
  Added shoulder_housing (fixed mount), upper_arm + shoulder_joint
  (revolute about body -y so positive = forward sweep), forearm +
  elbow_joint, end_effector (small green sphere). Both arm joints
  damping=0.005 friction=0.001 effort=2 vel=20.

src/drone.py
  Joint discovery in __post_init__ — finds shoulder_joint, elbow_joint,
  end_effector link by name. Initial pose set via resetJointState to
  folded (which is now == extended; see config note).

  ee_state(), gripper_world_position(), gripper_world_velocity() now
  query the EE link via p.getLinkState (was: fixed offset from base).
  joint_states() returns shoulder/elbow pos+vel for diagnostics.

  hold_arm/spin_arm/extend_arm/fold_arm convenience methods drive joint
  motors in POSITION_CONTROL or VELOCITY_CONTROL via setJointMotorControl2.
  step() now also calls _apply_arm() after the body force/torque application.

  grasp() attaches the held body to the END-EFFECTOR link (parentLinkIndex
  = ee_link) instead of the base. release() inherits gripper world velocity
  from getLinkState — handles arm rotation contribution implicitly.

  _system_com_world() computes the multi-body CoM summing base + all link
  masses. step() applies thrust at the system CoM (WORLD_FRAME with
  computed posObj) instead of the base origin (LINK_FRAME with [0,0,0]).
  Without this, articulating the arm shifts the CoM and creates a spurious
  pitch torque proportional to the offset — tested: arm extended fully
  forward used to drift drone 2 m and tilt 7.5° in 3 s; with CoM
  compensation, drift = 0.002 m, tilt = 0.7°.

  MASS bumped 0.55 → 0.625 to match URDF total (base 0.546 + 4 props 0.004
  + arm 0.075).

src/config.py
  ArmConfig dataclass: arm geometry (lengths, masses), motor limits, throw
  timing, release-trigger thresholds (multi-condition gates per plan §F).
  GameConfig.arm field.

  IMPORTANT NOTE in config: folded == extended (elbow=0). The intuitive
  "fold over" config (elbow=π) puts the EE+ball ABOVE the shoulder joint
  → inverted pendulum with √(g/L) ≈ 22 rad/s natural divergence rate.
  Joint motor PD can't stabilize it. Real hardware would fold via a
  different mechanism (e.g., sliding telescope or rotating into chassis);
  for sim we leave the arm always extended.

  floor_margin bumped 0.2 → 0.8 because extended arm (40 cm) plus PD
  overshoot (~30 cm) requires drone z to stay above ~0.8 m to keep ball
  off floor. play_area_min_offset.z adjusted accordingly.

src/controller.py
  max_thrust bumped 12 → 20 N (T/W ≈ 3.3, racing-class). The bowling
  throw with shrunken floor runway demands more thrust budget.

src/main.py
  Ball spawn at EE position (was: 8 cm below drone COM).
  snapshot() now logs shoulder_pos/vel, elbow_pos/vel, ee_pos, ee_vel
  for arm-aware diagnostics in check_run.py + plot_windup.py.

  THROW CHOREOGRAPHY rewritten as STATIONARY THROW for v1:
  - Drone hovers at planner's release_pos (no backup, no approach run).
  - Arm spin commanded at ω = |release_vel|/L (capped at URDF limit 18 rad/s).
  - Multi-condition release trigger from plan §F (min_spin_time gate +
    cos_align gate + (mag_met OR past_peak) trigger + safety timeout).
  - After release: refold arm, raise max_tilt for evade, go home.

  This is a SIMPLIFICATION of the planned bowling-style throw (drone
  runup + brake + arm spin combined). The full bowling version had too
  many simultaneous failure modes to debug in one session.

Current state: stationary throw fires reliably but EE world velocity is
~50% of planner's target_vel. Drone also drops/tilts during spin from
arm reaction torque. Catch fails. Not yet a working demo.

Next session: investigate why arm-tip velocity in world frame is half
the expected ω·L. Possible causes: drone falling during spin partially
cancels EE velocity; PyBullet's getLinkState may report something
different than expected; motor target velocity may not be the actual
joint velocity. Then re-introduce drone runup + brake to add the
translational+pitch contributions per the original bowling plan.

Co-Authored-By: Claude Opus 4.7 (1M context) <noreply@anthropic.com>

File: assets/quadrotor.urdf (robot description, URDF)
Before this commit: robot quadrotor, 5 links, 4 joints
Links:
- added link end_effector, mass 0.005; visual sphere radius=0.012
- added link forearm, mass 0.030; visual cylinder length=0.20 radius=0.008
- added link shoulder_housing, mass 0.010; visual cylinder length=0.020 radius=0.020
- added link upper_arm, mass 0.030; visual cylinder length=0.20 radius=0.008
Joints:
- added joint elbow_joint: type revolute, parent upper_arm, child forearm, origin xyz=0 0 -0.20, axis 0 1 0, limit lower=0 upper=3.2 effort=2.0 velocity=20
- added joint j_ee: type fixed, parent forearm, child end_effector, origin xyz=0 0 -0.20
- added joint j_shoulder_mount: type fixed, parent base_link, child shoulder_housing, origin xyz=0 0 0.030
- added joint shoulder_joint: type revolute, parent shoulder_housing, child upper_arm, origin xyz=0 0 -0.010, axis 0 -1 0, limit lower=-100 upper=100 effort=2.0 velocity=20
