Commit message: M8: real caging gripper (4x3-segment, long proximal) on the catcher
The 2-segment fingers only CONTAINED a ball in an upright cup (failed the
inversion test, §13). Fixed with the user's design: 4 fingers x 3 segments
with a long proximal phalanx (human-like) — proximal reaches the ball's
equator, middle+distal curl under to meet beneath it (form closure that
survives full 180deg inversion).

Productionized:
- make_gripper_urdf.py generalized to N-segment fingers (finger{i}_seg{k});
  default 4 fingers x 3 segments, SEG_LENS=(55,32,25)mm, MOUNT_R=34mm.
- Drone finger API: finger_joints is now per-finger segment lists; open/close
  drive per-segment angle tuples (config.finger_open/finger_close).
- Hover-stability fix: 12 PD finger joints on a floating base overwhelm the
  contact solver (body diverges ~80cm). Pin fingers kinematically while OPEN
  (resetJointState), motorize only to close -> 1.2cm hover; elbow_catch_solo
  also bumps numSolverIterations=150. The §13 yaw singularity does not recur.

Validated on the drone: hovers stable, 4 fingers close on a ball, held
through a 30cm lift (static ball).

Dynamic catch (elbow_catch_solo with the new hand): IK tracking puts the cup
on the ball to ~2cm and all 4 fingers contact, but does NOT yet retain — the
ball arrives at ~2.3 m/s relative and punches through before the cage firms.
Position tracking is solved; VELOCITY MATCHING is the single remaining piece
(Jacobian joint-velocity control so the cup moves with the ball at contact).

No regression: arm_catch_solo --grid still 12/12; plain drone mass 0.625.

Docs: iteration_findings §15, concepts/09 (force vs form closure, screenshot
review caught the bug, N-PD-joints solver instability), CLAUDE.md (modules,
test entry, parking lot #2-3).

Co-Authored-By: Claude Opus 4.8 (1M context) <noreply@anthropic.com>

File: assets/quadrotor_gripper.urdf (robot description, URDF)
Before this commit: robot quadrotor_gripper, 15 links, 14 joints
Links:
- removed link finger0_dist
- removed link finger0_prox
- removed link finger1_dist
- removed link finger1_prox
- removed link finger2_dist
- removed link finger2_prox
- added link finger0_seg0, mass 0.004; collision box size=0.014 0.014 0.055; visual box size=0.014 0.014 0.055
- added link finger0_seg1, mass 0.0035; collision box size=0.014 0.014 0.032; visual box size=0.014 0.014 0.032
- added link finger0_seg2, mass 0.003; collision box size=0.014 0.014 0.025; visual box size=0.014 0.014 0.025
- added link finger1_seg0, mass 0.004; collision box size=0.014 0.014 0.055; visual box size=0.014 0.014 0.055
- added link finger1_seg1, mass 0.0035; collision box size=0.014 0.014 0.032; visual box size=0.014 0.014 0.032
- added link finger1_seg2, mass 0.003; collision box size=0.014 0.014 0.025; visual box size=0.014 0.014 0.025
- added link finger2_seg0, mass 0.004; collision box size=0.014 0.014 0.055; visual box size=0.014 0.014 0.055
- added link finger2_seg1, mass 0.0035; collision box size=0.014 0.014 0.032; visual box size=0.014 0.014 0.032
- added link finger2_seg2, mass 0.003; collision box size=0.014 0.014 0.025; visual box size=0.014 0.014 0.025
- added link finger3_seg0, mass 0.004; collision box size=0.014 0.014 0.055; visual box size=0.014 0.014 0.055
- added link finger3_seg1, mass 0.0035; collision box size=0.014 0.014 0.032; visual box size=0.014 0.014 0.032
- added link finger3_seg2, mass 0.003; collision box size=0.014 0.014 0.025; visual box size=0.014 0.014 0.025
Joints:
- removed joint finger0_dist_joint
- removed joint finger0_prox_joint
- removed joint finger1_dist_joint
- removed joint finger1_prox_joint
- removed joint finger2_dist_joint
- removed joint finger2_prox_joint
- added joint finger0_seg0_joint: type revolute, parent forearm, child finger0_seg0, origin xyz=0.0000 0.0340 -0.20, axis -1.0000 0.0000 0, limit lower=-0.8 upper=2.0 effort=0.6 velocity=15
- added joint finger0_seg1_joint: type revolute, parent finger0_seg0, child finger0_seg1, origin xyz=0 0 -0.0550, axis -1.0000 0.0000 0, limit lower=-0.8 upper=2.0 effort=0.6 velocity=15
- added joint finger0_seg2_joint: type revolute, parent finger0_seg1, child finger0_seg2, origin xyz=0 0 -0.0320, axis -1.0000 0.0000 0, limit lower=-0.8 upper=2.0 effort=0.6 velocity=15
- added joint finger1_seg0_joint: type revolute, parent forearm, child finger1_seg0, origin xyz=-0.0340 0.0000 -0.20, axis -0.0000 -1.0000 0, limit lower=-0.8 upper=2.0 effort=0.6 velocity=15
- added joint finger1_seg1_joint: type revolute, parent finger1_seg0, child finger1_seg1, origin xyz=0 0 -0.0550, axis -0.0000 -1.0000 0, limit lower=-0.8 upper=2.0 effort=0.6 velocity=15
- added joint finger1_seg2_joint: type revolute, parent finger1_seg1, child finger1_seg2, origin xyz=0 0 -0.0320, axis -0.0000 -1.0000 0, limit lower=-0.8 upper=2.0 effort=0.6 velocity=15
- added joint finger2_seg0_joint: type revolute, parent forearm, child finger2_seg0, origin xyz=-0.0000 -0.0340 -0.20, axis 1.0000 -0.0000 0, limit lower=-0.8 upper=2.0 effort=0.6 velocity=15
- added joint finger2_seg1_joint: type revolute, parent finger2_seg0, child finger2_seg1, origin xyz=0 0 -0.0550, axis 1.0000 -0.0000 0, limit lower=-0.8 upper=2.0 effort=0.6 velocity=15
- added joint finger2_seg2_joint: type revolute, parent finger2_seg1, child finger2_seg2, origin xyz=0 0 -0.0320, axis 1.0000 -0.0000 0, limit lower=-0.8 upper=2.0 effort=0.6 velocity=15
- added joint finger3_seg0_joint: type revolute, parent forearm, child finger3_seg0, origin xyz=0.0340 -0.0000 -0.20, axis 0.0000 1.0000 0, limit lower=-0.8 upper=2.0 effort=0.6 velocity=15
- added joint finger3_seg1_joint: type revolute, parent finger3_seg0, child finger3_seg1, origin xyz=0 0 -0.0550, axis 0.0000 1.0000 0, limit lower=-0.8 upper=2.0 effort=0.6 velocity=15
- added joint finger3_seg2_joint: type revolute, parent finger3_seg1, child finger3_seg2, origin xyz=0 0 -0.0320, axis 0.0000 1.0000 0, limit lower=-0.8 upper=2.0 effort=0.6 velocity=15
